File: HW/SensorBoard.sch (EAGLE design)
At the start: 24 parts, among them U1 ATMEGA328P_TQFP, X1 16mhz, X2 49S/18PF

Commit message: V1.0
Parts:
- removed C6: 100uf, rcl:CPOL-EU153CLV-0505
- added C5: 100uf, rcl:C-EUC1206
- added SW: (no value), adafruit:SWITCH_PUSHBUTTONC&K_KSS
- SW1: device adafruit:SWITCH_PUSHBUTTONC&K_KSS -> SparkFun-Switches:MOMENTARY-SWITCH-SPST-2-SMD-5.2MM
- UART: device pinhead:PINHD-1X2 -> pinhead:PINHD-1X4
- X1: value 16mhz -> 7B-16.000MAAJ-T; device Crystals:FC4SDCBMF16.0-T1 -> Crystals:7B-16.000MAAJ-T
- X2: value 49S/18PF -> FC4SDCBMF16.0-T1; device Crystals:49S/18PF -> Crystals:FC4SDCBMF16.0-T1
Connections:
- new net ADDR_SENSE: U1.PC1(ADC1), UART.3
- net +5V: now also C5.1; no longer C6.+
- net GND: now also C5.2, SW.P$2, SW1.3, SW1.4, UART.4; no longer C6.-, SW1.P$2
- net N$1: now also X1.3; no longer X1.1
- net N$2: now also X1.1; no longer X1.2
- net RESET: now also SW.P$1, SW1.1, SW1.2; no longer SW1.P$1
Other:
- moved on the sheet: C3, R3, X2

Commit message: adding signalisation leds
Parts:
- added LED1: POWER, led:LEDSMT1206
- added LED2: STATUS, led:LEDSMT1206
- added R4, R5: 1K, rcl:R-EU_M1206
Connections:
- new net N$3: LED2.A, R4.1
- new net N$4: LED1.A, R5.1
- new net STATUS: LED2.C, U1.PC0(ADC0)
- net +5V: now also LED1.C
- net GND: now also R4.2, R5.2
