File: HW/SensorBoard.sch (EAGLE design)
At the start: 29 parts, among them U1 ATMEGA328P_TQFP, X1 7B-16.000MAAJ-T, X2 FC4SDCBMF16.0-T1

Commit message: commit
Connections:
- net S_A: now also U1.ADC6
Changed lines of the file:
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@@
 <label x="195.58" y="58.42" size="1.778" layer="95" rot="R180" xref="yes"/>
+</segment>
+<segment>
+<pinref part="U1" gate="U$1" pin="ADC6"/>
+<wire x1="165.1" y1="71.12" x2="167.64" y2="71.12" width="0.1524" layer="91"/>
+<label x="167.64" y="71.12" size="1.778" layer="95" xref="yes"/>
 </segment>
 </net>
