File: HW/SensorBoard.brd (EAGLE design)
At the start: 50 x 50 mm, 29 parts, among them U1 ATMEGA328P_TQFP, X1 7B-16.000MAAJ-T, X2 FC4SDCBMF16.0-T1

Commit message: commit
Connections:
- net S_A: now also U1.19
Routing:
- net S_A: track 9.12 -> 21.9 mm, vias 0 -> 1
- net S_TX: track 30.0 -> 30.5 mm
Changed lines of the file:
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@@
 </layers>
 <board>
-<fusionsync huburn="a.cGVyc29uYWw6dWUyOTc5YzVj" projecturn="a.cGVyc29uYWw6dWUyOTc5YzVjIzIwMjAwNzEyMzE1MTM4MDI2" f3durn="urn:adsk.wipprod:dm.lineage:Zer31BQvS1-_2MtQUhH37g" pcbguid="b9daa228-3daa-436f-8b60-8e0eecd0a705" lastpulledtime="" lastsyncedchangeguid="beda2d17-c0b7-454d-79ff-fd73764223b2"/>
+<fusionsync huburn="a.cGVyc29uYWw6dWUyOTc5YzVj" projecturn="a.cGVyc29uYWw6dWUyOTc5YzVjIzIwMjAwNzEyMzE1MTM4MDI2" f3durn="urn:adsk.wipprod:dm.lineage:Zer31BQvS1-_2MtQUhH37g" pcbguid="b9daa228-3daa-436f-8b60-8e0eecd0a705" lastpulledtime="" lastsyncedchangeguid="374a7302-eaff-bae3-b5fb-a31393b8b76e"/>
 <plain>
 <wire x1="-20" y1="-25" x2="20" y2="-25" width="0" layer="20"/>
@@
 <wire x1="2.8" y1="4.2926" x2="2.8" y2="2.8" width="0.254" layer="1"/>
 <via x="2.8" y="2.8" extent="1-16" drill="0.35"/>
-<wire x1="-11.094" y1="3.175" x2="2.425" y2="3.175" width="0.254" layer="16"/>
-<wire x1="2.425" y1="3.175" x2="2.8" y2="2.8" width="0.254" layer="16"/>
 <wire x1="-11.094" y1="10.126" x2="-11.1" y2="10" width="0.254" layer="1"/>
 <wire x1="-11.094" y1="3.175" x2="-11.094" y2="10.126" width="0.254" layer="1"/>
 <via x="2.6424" y="-1.7" extent="1-16" drill="0.35"/>
-<wire x1="4.2926" y1="-2.8" x2="4.0514" y2="-2.5588" width="0.254" layer="1"/>
-<wire x1="4.0514" y1="-2.5588" x2="3.54186875" y2="-2.5588" width="0.254" layer="1"/>
-<wire x1="2.68306875" y1="-1.7" x2="2.6424" y2="-1.7" width="0.254" layer="1"/>
-<wire x1="3.54186875" y1="-2.5588" x2="2.68306875" y2="-1.7" width="0.254" layer="1"/>
+<wire x1="2.6424" y1="-1.7" x2="2.68306875" y2="-1.7" width="0.254" layer="1"/>
 <wire x1="2.6424" y1="-1.7" x2="2.4682" y2="-1.5258" width="0.254" layer="16"/>
 <wire x1="2.4682" y1="-1.5258" x2="2.4682" y2="0.1" width="0.254" layer="16"/>
@@
 <wire x1="2.4682" y1="0.1" x2="1.8" y2="0.7682" width="0.254" layer="1"/>
 <wire x1="1.8" y1="1.8" x2="2.8" y2="2.8" width="0.254" layer="1"/>
+<wire x1="-11.094" y1="3.175" x2="-10.469" y2="3.8" width="0.254" layer="16"/>
+<wire x1="1.8" y1="3.8" x2="2.8" y2="2.8" width="0.254" layer="16"/>
+<wire x1="-10.469" y1="3.8" x2="1.8" y2="3.8" width="0.254" layer="16"/>
+<wire x1="3.78306875" y1="-2.8" x2="4.2926" y2="-2.8" width="0.254" layer="1"/>
+<wire x1="2.68306875" y1="-1.7" x2="3.78306875" y2="-2.8" width="0.254" layer="1"/>
 </signal>
 <signal name="GND">
@@
 <contactref element="U1" pad="2"/>
 <via x="1.8" y="-0.8" extent="1-16" drill="0.35"/>
-<wire x1="3.78306875" y1="-2" x2="3.3" y2="-1.51693125" width="0.254" layer="1"/>
-<wire x1="3.3" y1="-1.51693125" x2="3.3" y2="-1" width="0.254" layer="1"/>
-<wire x1="3.15" y1="-0.85" x2="3.3" y2="-1" width="0.254" layer="1"/>
+<wire x1="3.3" y1="-1.51693125" x2="3.78306875" y2="-2" width="0.254" layer="1"/>
+<wire x1="3.3" y1="-1.3" x2="3.3" y2="-1.51693125" width="0.254" layer="1"/>
 <wire x1="3.78306875" y1="-2" x2="4.2926" y2="-2" width="0.254" layer="1"/>
 <wire x1="-8.554" y1="1.905" x2="-7.0245" y2="0.3755" width="0.254" layer="16"/>
 <wire x1="-7.0245" y1="0.3755" x2="0.6245" y2="0.3755" width="0.254" layer="16"/>
 <wire x1="0.6245" y1="0.3755" x2="1.8" y2="-0.8" width="0.254" layer="16"/>
-<wire x1="3.15" y1="-0.85" x2="1.85" y2="-0.85" width="0.254" layer="1"/>
 <wire x1="1.85" y1="-0.85" x2="1.8" y2="-0.8" width="0.254" layer="1"/>
 <wire x1="1.8" y1="-0.8" x2="1.8" y2="-2.6" width="0.254" layer="1"/>
 <wire x1="1.8" y1="-2.6" x2="2.8" y2="-3.6" width="0.254" layer="1"/>
 <wire x1="2.8" y1="-3.6" x2="2.8" y2="-4.2926" width="0.254" layer="1"/>
+<wire x1="3.3" y1="-1.3" x2="2.85" y2="-0.85" width="0.254" layer="1"/>
+<wire x1="2.85" y1="-0.85" x2="2.6" y2="-0.85" width="0.254" layer="1"/>
+<wire x1="2.6" y1="-0.85" x2="1.85" y2="-0.85" width="0.254" layer="1"/>
 </signal>
 <signal name="+5V">
@@
 <wire x1="-14.1" y1="-10" x2="-8.554" y2="-4.454" width="0.254" layer="1"/>
 <wire x1="-8.554" y1="-4.454" x2="-8.554" y2="-3.175" width="0.254" layer="1"/>
+<contactref element="U1" pad="19"/>
+<via x="-5.907259375" y="1.692740625" extent="1-16" drill="0.35"/>
+<wire x1="-4.2926" y1="1.2" x2="-5.41451875" y2="1.2" width="0.254" layer="1"/>
+<wire x1="-5.41451875" y1="1.2" x2="-5.907259375" y2="1.692740625" width="0.254" layer="1"/>
+<wire x1="-5.907259375" y1="1.692740625" x2="-7.21451875" y2="3" width="0.254" layer="16"/>
+<wire x1="-9.3" y1="3" x2="-9.9" y2="2.4" width="0.254" layer="16"/>
+<wire x1="-9.9" y1="2.4" x2="-9.9" y2="-1.829" width="0.254" layer="16"/>
+<wire x1="-9.9" y1="-1.829" x2="-8.554" y2="-3.175" width="0.254" layer="16"/>
+<wire x1="-7.21451875" y1="3" x2="-9.3" y2="3" width="0.254" layer="16"/>
 </signal>
 <signal name="SDA">
@@
 <contactref element="U1" pad="23"/>
 <via x="-5" y="-5" extent="1-16" drill="0.35"/>
-<wire x1="-3.54186875" y1="-2.2412" x2="-3.3782" y2="-2.40486875" width="0.254" layer="1"/>
-<wire x1="-4.2926" y1="-2" x2="-4.0514" y2="-2.2412" width="0.254" layer="1"/>
-<wire x1="-4.0514" y1="-2.2412" x2="-3.54186875" y2="-2.2412" width="0.254" layer="1"/>
 <wire x1="-3.3782" y1="-2.40486875" x2="-3.3782" y2="-3.3782" width="0.254" layer="1"/>
 <wire x1="-3.3782" y1="-3.3782" x2="-5" y2="-5" width="0.254" layer="1"/>
@@
 <wire x1="-6" y1="-8" x2="-6" y2="-9.528" width="0.254" layer="1"/>
 <wire x1="-6" y1="-9.528" x2="-5.95" y2="-9.578" width="0.254" layer="1"/>
+<wire x1="-4.2926" y1="-2" x2="-3.78306875" y2="-2" width="0.254" layer="1"/>
+<wire x1="-3.78306875" y1="-2" x2="-3.3782" y2="-2.40486875" width="0.254" layer="1"/>
 </signal>
 </signals>
 <mfgpreviewcolors>
-<mfgpreviewcolor name="soldermaskcolor" color="0xC8008000"/>
-<mfgpreviewcolor name="silkscreencolor" color="0xFFFEFEFE"/>
+<mfgpreviewcolor name="soldermaskcolor" color="0xC8FCFCFC"/>
+<mfgpreviewcolor name="silkscreencolor" color="0xFF000000"/>
 <mfgpreviewcolor name="backgroundcolor" color="0xFF282828"/>
-<mfgpreviewcolor name="coppercolor" color="0xFFFFBF00"/>
+<mfgpreviewcolor name="coppercolor" color="0xFFBCBCBC"/>
 <mfgpreviewcolor name="substratecolor" color="0xFF786E46"/>
 </mfgpreviewcolors>
