File: HW/ControlBoard/Controlboard.brd (EAGLE design)
At the start: 50 x 50 mm, 38 parts, among them Q1 BSS138, U1 MPU-6050MPU6050, X1 B4B-ZR, X2 B4B-ZR, X3 B4B-ZR, X4 B4B-ZR, X5 B4B-ZR, X6 B4B-ZR, X8 B4B-ZR

Commit message: commit
Parts:
- removed X1, X2, X3, X4, X5, X6, X8: B4B-ZR, con-jst:B4B-ZR
- added JP2, JP3, JP4, JP5: (no value), pinhead:1X04
- moved R7 0.15 mm to (10.3, 3.80)
Connections:
- net +5V: now also JP2.1, JP3.1, JP4.1, JP5.1; no longer X1.1, X2.1, X3.1, X4.1, X5.1, X6.1, X8.1
- net A0: now also JP2.2; no longer X8.2
- net A1: now also JP2.3; no longer X8.3
- net GND: now also JP2.4, JP3.4, JP4.4, JP5.4; no longer X1.4, X2.4, X3.4, X4.4, X5.4, X6.4, X8.4
- net SCL: now also JP3.3, JP4.3, JP5.3; no longer X1.3, X2.3, X3.3, X4.3, X5.3, X6.3
- net SDA: now also JP3.2, JP4.2, JP5.2; no longer X1.2, X2.2, X3.2, X4.2, X5.2, X6.2
Routing:
- net +5V: track 45.3 -> 69.8 mm
- net SCL: track 87.2 -> 74.3 mm
- net BT_RX: track 23.8 -> 15.0 mm
- net GND: track 32.8 -> 24.4 mm
- net A0: track 30.9 -> 36.2 mm
- net A1: track 35.5 -> 39.6 mm
Other:
- board text removed: "+5V SDA SCL GND"
