File: HW/ControlBoard/Controlboard.sch (EAGLE design)
At the start: 38 parts, among them Q1 BSS138, U1 MPU-6050MPU6050, X1 B4B-ZR, X2 B4B-ZR, X3 B4B-ZR, X4 B4B-ZR, X5 B4B-ZR, X6 B4B-ZR, X8 B4B-ZR

Commit message: commit
Parts:
- removed X1, X2, X3, X4, X5, X6, X8: B4B-ZR, con-jst:B4B-ZR
- added JP2, JP3, JP4, JP5: (no value), pinhead:PINHD-1X4
Connections:
- net +5V: now also JP2.1, JP3.1, JP4.1, JP5.1; no longer X1-1.1, X2-1.1, X3-1.1, X4-1.1, X5-1.1, X6-1.1, X8-1.1
- net A0: now also JP2.2; no longer X8-2.1
- net A1: now also JP2.3; no longer X8-3.1
- net GND: now also JP2.4, JP3.4, JP4.4, JP5.4; no longer X1-4.1, X2-4.1, X3-4.1, X4-4.1, X5-4.1, X6-4.1, X8-4.1
- net SCL: now also JP3.3, JP4.3, JP5.3; no longer X1-3.1, X2-3.1, X3-3.1, X4-3.1, X5-3.1, X6-3.1
- net SDA: now also JP3.2, JP4.2, JP5.2; no longer X1-2.1, X2-2.1, X3-2.1, X4-2.1, X5-2.1, X6-2.1
